File: pcb/vera-module.brd (EAGLE design)
At the start: 69.8 x 48.3 mm, 102 parts, among them J1 VIDEO, J2 BOOT0, J3 HDR8X1, J4 BUS, J5 HDR8X1, J6 5V_OUT, J7 10118193-0001LF, J8 SWD, J9 SERIAL, U1 ICE40UP5K-SG48ITR50, U10 STM32F070F6P6, U11 TC1185-3.3VCT713, U2 THS7314D, U3 SN74CBTD3861PWR, U4 W25Q16JVSNIQ, U5 SG5032CAN_25.000000M-TJGA3, U6 74LVC4245APW, U7 AP3417CKTR-G1, U8 AP3417CKTR-G1, U9 74AHCT1G14SE-7, X2 7A-8.000MAAE-T

Commit message: Fixes for release to Kevin.
Parts:
- R28, R29: value 499 -> 1.2k
- R33: value 75 -> 0
Changed lines of the file:
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@@
 <element name="R27" library="rcl" package="R0603" value="60.4k" x="57.78" y="39.65" rot="R90"/>
 <element name="R2" library="rcl" package="R0603" value="9.31k" x="44.98" y="39.65" rot="R90"/>
-<element name="R28" library="rcl" package="R0603" value="499" x="43.43" y="39.65" rot="R270"/>
-<element name="R29" library="rcl" package="R0603" value="499" x="59.38" y="39.65" rot="R270"/>
+<element name="R28" library="rcl" package="R0603" value="1.2k" x="43.43" y="39.65" rot="R270"/>
+<element name="R29" library="rcl" package="R0603" value="1.2k" x="59.38" y="39.65" rot="R270"/>
 <element name="U2" library="integrated_circuits" package="SOIC-8" value="THS7314D" x="38.13" y="35" rot="R90"/>
 <element name="R30" library="rcl" package="R0603" value="75" x="40.93" y="43.3" rot="R90"/>
@@
 <element name="C2" library="rcl" package="C0805" value="10u" x="43.43" y="33.2" rot="R270"/>
 <element name="C3" library="rcl" package="C0603" value="1n" x="37.83" y="43.3" rot="R90"/>
-<element name="R33" library="rcl" package="R0603" value="75" x="38.58" y="40.95" rot="R180"/>
+<element name="R33" library="rcl" package="R0603" value="0" x="38.58" y="40.95" rot="R180"/>
 <element name="U3" library="integrated_circuits" package="TSSOP-24" value="SN74CBTD3861PWR" x="57.13" y="10.5" rot="R270"/>
 <element name="R34" library="rcl" package="R0603" value="10k" x="48.83" y="32.2"/>
