File: pcb/vera-module.sch (EAGLE design)
At the start: 102 parts, among them J1 VIDEO, J2 BOOT0, J3 HDR8X1, J4 BUS, J5 HDR8X1, J6 5V_OUT, J7 10118193-0001LF, J8 SWD, J9 SERIAL, U1 ICE40UP5K-SG48ITR50, U10 STM32F070F6P6, U11 TC1185-3.3VCT713, U2 THS7314D, U3 SN74CBTD3861PWR, U4 W25Q16JVSNIQ, U5 SG5032CAN_25.000000M-TJGA3, U6 74LVC4245APW, U7 AP3417CKTR-G1, U8 AP3417CKTR-G1, U9 74AHCT1G14SE-7, X2 7A-8.000MAAE-T

Commit message: Fixes for release to Kevin.
Parts:
- R28, R29: value 499 -> 1.2k
- R33: value 75 -> 0
Changed lines of the file:
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@@
 <part name="R2" library="rcl" deviceset="RESISTOR" device="0603" value="9.31k"/>
 <part name="U$2" library="supply" deviceset="GND" device=""/>
-<part name="R28" library="rcl" deviceset="RESISTOR" device="0603" value="499"/>
-<part name="R29" library="rcl" deviceset="RESISTOR" device="0603" value="499"/>
+<part name="R28" library="rcl" deviceset="RESISTOR" device="0603" value="1.2k"/>
+<part name="R29" library="rcl" deviceset="RESISTOR" device="0603" value="1.2k"/>
 <part name="U$3" library="supply" deviceset="GND" device=""/>
 <part name="U$4" library="supply" deviceset="GND" device=""/>
@@
 <part name="GND1" library="supply" deviceset="GND" device=""/>
 <part name="C3" library="rcl" deviceset="CAPACITOR" device="0603" value="1n"/>
-<part name="R33" library="rcl" deviceset="RESISTOR" device="0603" value="75"/>
+<part name="R33" library="rcl" deviceset="RESISTOR" device="0603" value="0"/>
 <part name="U$27" library="supply" deviceset="GND" device=""/>
 <part name="U3" library="integrated_circuits" deviceset="SN74CBTD3861PWR" device=""/>
